File: iso9141-interface.kicad_sch (KiCad schematic)
At the start: 19 parts, among them J1 Conn_01x03, J2 Conn_01x05, Q1 MMBT3904, Q2 MMBT3904, Q3 MMBT3904

Commit message: Commiting V2 files that were previously missing
Other:
- title: (none) -> ISO9141 Interface Board
Changed lines of the file:
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@@
 (kicad_sch (version 20230121) (generator eeschema)
-  (paper "A4")
+  (paper "USLetter")
+  (title_block
+    (title "ISO9141 Interface Board")
+  )
   (junction (at 90.17 81.28) (diameter 0) (color 0 0 0 0)
   )
